File: KiCAD_MCPtest/KiCAD_MCPtest.kicad_sch (KiCad schematic)
At the start: 72 parts, among them J1 Conn_01x04, J2 Conn_01x04, J3 Conn_01x05, J4 Conn_01x04, J5 Conn_01x05, J6 Conn_01x04, P1 USB_C_Plug_USB2.0, U1 STM32F103C8Tx, U2 MCP2562-E-SN, U3 MP2359DJ-LF-Z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

Commit message: PCB made
Parts:
- removed P1: USB_C_Plug_USB2.0, Connector_USB:USB_C_Receptacle_Palconn_UTC16-G, symbol Connector:USB_C_Plug_USB2.0
- removed R10, R2: 10k, Resistor_SMD:R_0402_1005Metric, symbol Device:R_Small
- added F1: 500mA, Fuse:Fuse_0603_1608Metric, symbol Device:Fuse_Small
- added J7: USB_C, Connector:USB_C_HRO_TYPE-C-31-M-12, symbol Connector:USB_C_Receptacle_USB2.0_14P
- added R20, R21: 5.1k, Resistor_SMD:R_0402_1005Metric, symbol Device:R_Small
- added R22: 10k, Resistor_SMD:R_0402_1005Metric, symbol Device:R_Small
- added SW1: SW_Push, Button_Switch_SMD:Button_TL3342, symbol Switch:SW_Push
Connections:
- net +3V3: now also SW1.1
- net +5V: now also F1.2
- net GND: now also J7.A1 (GND), J7.A12 (GND), J7.B1 (GND), J7.B12 (GND), J7.S1 (SHIELD), R20.2, R21.2, R22.1
- net USB_CONN_D+: now also J7.A6 (D+), J7.B6 (D+)
- net USB_CONN_D-: now also J7.A7 (D-), J7.B7 (D-)
- net BOOT0: now reaches U1.44 (BOOT0)
- net BOOT0: now also R22.2, SW1.2
- new net: F1.1, J7.A4 (VBUS), J7.A9 (VBUS), J7.B4 (VBUS), J7.B9 (VBUS)
- new net: J7.A5 (CC1), R20.1
- new net: J7.B5 (CC2), R21.1
- no-connect marks 53 -> 52

Commit message: pcb ordered
Parts:
- D1, D4: LCSC Part # C72041 -> C2286
- D2: LCSC Part # C8598 -> C64885
- F1: LCSC C210357 -> (none); LCSC Part # (none) -> C210357
- J7: LCSC C165948 -> (none); LCSC Part # (none) -> C165948
- L1, L3: LCSC Part # C26443 -> C395063
- R20, R21: LCSC C25905 -> (none); LCSC Part # (none) -> C25905
- R22: LCSC C25744 -> (none); LCSC Part # (none) -> C25744
- SW1: LCSC C115351 -> (none); LCSC Part # (none) -> C115351
- U2, U4: LCSC Part # C53609 -> C124016
- U3: LCSC Part # C14259 -> C18198375
