File: KiCAD_MCPtest/KiCAD_MCPtest.kicad_pcb (KiCad board)
At the start: 4 copper layers, 60 x 65 mm, 72 parts, among them J1 Conn_01x04, J2 Conn_01x04, J3 Conn_01x05, J4 Conn_01x04, J5 Conn_01x05, J6 Conn_01x04, P1 USB_C_Plug_USB2.0, U1 STM32F103C8Tx, U2 MCP2562-E-SN, U3 MP2359DJ-LF-Z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

Commit message: PCB made
Parts:
- removed P1: USB_C_Plug_USB2.0, Connector_USB:USB_C_Receptacle_Palconn_UTC16-G
- removed R10, R2: 10k, Resistor_SMD:R_0402_1005Metric
- added F1: 500mA, Fuse:Fuse_0603_1608Metric, F.Cu at (125.6, 96.8)
- added J7: USB_C, Connector:USB_C_HRO_TYPE-C-31-M-12, F.Cu at (120.6, 104.8)
- added R20: 5.1k, Resistor_SMD:R_0402_1005Metric, F.Cu at (112.2, 100.4)
- added R21: 5.1k, Resistor_SMD:R_0402_1005Metric, F.Cu at (112.2, 102.6)
- added R22: 10k, Resistor_SMD:R_0402_1005Metric, F.Cu at (123.5, 56.5)
- added SW1: SW_Push, Button_Switch_SMD:Button_TL3342, F.Cu at (130.1, 56.2)
- C13: value 10n -> 10nF
- L2: value 10u -> 10uH
Connections:
- U1 pad 44: Net-(U1-BOOT0) -> BOOT0
Routing:
- net BOOT0: track 0.00 -> 24.3 mm, vias 0 -> 2
- net Net-(J7-CC2): track 0.00 -> 12.1 mm
- net Net-(F1-Pad1): track 0.00 -> 11.5 mm, vias 0 -> 2
- net Net-(J7-CC1): track 0.00 -> 9.45 mm
- net Net-(U1-BOOT0): track 9.00 -> 0.00 mm
- net GND: track 76.7 -> 68.6 mm, vias 46 -> 49
- net +3V3: track 59.9 -> 68.0 mm, vias 20 -> 21
- net Net-(P1-CC): track 6.54 -> 0.00 mm
- net +5V: track 17.4 -> 11.0 mm
- net USB_CONN_D-: track 8.38 -> 10.7 mm, vias 2 -> 0
- net USB_CONN_D+: track 8.55 -> 10.7 mm
- net I2C1_SDA: track 57.9 -> 57.2 mm

Commit message: save
Routing:
- net GND: track 68.6 -> 64.5 mm
Changed lines of the file:
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@@
 		(property "Reference" "H1"
 			(at 0 5.5 0)
-			(layer "F.SilkS")
+			(layer "F.Fab")
 			(effects
 				(font
@@
 		(property "Reference" "H3"
 			(at 0 -5.3 0)
-			(layer "F.SilkS")
+			(layer "F.Fab")
 			(effects
 				(font
@@
 		(tags "resistor")
 		(property "Reference" "R20"
-			(at -0.01 1.3 360)
+			(at -0.01 1.3 0)
 			(layer "F.SilkS")
 			(effects
@@
 		)
 		(property "Value" "5.1k"
-			(at 0 1.17 360)
+			(at 0 1.17 0)
 			(layer "F.Fab")
 			(effects
@@
 		)
 		(fp_text user "${REFERENCE}"
-			(at 0 0 360)
+			(at 0 0 0)
 			(layer "F.Fab")
 			(effects
@@
 		(property "Reference" "H2"
 			(at 0 5.5 0)
-			(layer "F.SilkS")
+			(layer "F.Fab")
 			(effects
 				(font
@@
 		(property "Reference" "H4"
 			(at 0 -5.3 0)
-			(layer "F.SilkS")
+			(layer "F.Fab")
 			(effects
 				(font
@@
 		(tags "resistor")
 		(property "Reference" "R21"
-			(at 0 -1.3 360)
+			(at 0 -1.3 0)
 			(layer "F.SilkS")
 			(effects
@@
 		)
 		(property "Value" "5.1k"
-			(at 0 1.17 360)
+			(at 0 1.17 0)
 			(layer "F.Fab")
 			(effects
@@
 		)
 		(fp_text user "${REFERENCE}"
-			(at 0 0 360)
+			(at 0 0 0)
 			(layer "F.Fab")
 			(effects
@@
 	)
 	(segment
-		(start 116 63.7)
-		(end 115.1 62.8)
-		(width 0.5)
-		(layer "F.Cu")
-		(net 2)
-	)
-	(segment
 		(start 131.15 72.65)
 		(end 130.8 73)
@@
 	)
 	(segment
-		(start 113.870001 62.8)
-		(end 112.99 63.680001)
-		(width 0.5)
-		(layer "F.Cu")
-		(net 2)
-	)
-	(segment
 		(start 146.25 68.25)
 		(end 144.6625 68.25)
@@
 	)
 	(segment
-		(start 115.1 62.8)
-		(end 113.870001 62.8)
-		(width 0.5)
-		(layer "F.Cu")
-		(net 2)
-	)
-	(segment
 		(start 143 61.6)
 		(end 143 61.02)
@@
 		(width 0.5)
 		(layer "F.Cu")
-		(net 2)
-	)
-	(segment
-		(start 112.99 63.680001)
-		(end 112.99 64)
-		(width 0.5)
-		(layer "F.Cu")
